File: bms_slave.kicad_pcb (KiCad board)
At the start: 4 copper layers, 75 x 45 mm, 120 parts, among them J1 0436500218, J2 0430450212, J3 0430451612, J4 0430451200, J4 0436501200, Q1 ZXTN4004KQTC, U1 BQ79616PAPRQ1, U2 SM91502ALA-E, U3 SM91502ALA-E

Commit message: PCB[Dasiy, Sens, Bal]:Added clearnece rules for pad to Daisy, 3W for Daisy, Via shield, started routing for bal and sens.
Parts:
- moved C20 3.58 mm to (143.8, 98.8)
- moved C19 3.53 mm to (142.3, 100.3)
- moved C17 3.46 mm to (139.2, 100.3)
- moved C18 3.46 mm to (140.7, 98.8)
- moved C16 3.41 mm to (137.6, 98.8)
- moved C15 3.36 mm to (136.1, 100.3)
- moved C14 3.31 mm to (134.5, 98.8)
- moved C13 3.26 mm to (133.0, 100.3)
- moved C4 3.18 mm to (131.4, 98.8)
- moved C3 3.13 mm to (129.9, 100.3)
- moved C1 0.08 mm to (128.3, 98.8)
Routing:
- net /Project Architecture/Cell Sense & Balance/CB7: track 0.00 -> 6.42 mm, vias 0 -> 1
- net /Project Architecture/Cell Sense & Balance/CB1: track 0.00 -> 5.22 mm, vias 0 -> 1
- net /Project Architecture/Cell Sense & Balance/CB2: track 0.00 -> 4.93 mm, vias 0 -> 1
- net /Project Architecture/Cell Sense & Balance/CB6: track 0.00 -> 4.88 mm, vias 0 -> 1
- net /Project Architecture/Cell Sense & Balance/CB3: track 0.00 -> 4.70 mm, vias 0 -> 1
- net /Project Architecture/Cell Sense & Balance/CB5: track 0.00 -> 4.66 mm, vias 0 -> 1
- net /Project Architecture/Cell Sense & Balance/CB4: track 0.00 -> 4.47 mm, vias 0 -> 1
- net /Project Architecture/Cell Sense & Balance/CB0: track 1.47 -> 5.01 mm, vias 1 -> 3
- net /Project Architecture/Cell Sense & Balance/VC5: track 34.9 -> 38.2 mm
- net /Project Architecture/Cell Sense & Balance/VC2: track 28.4 -> 31.6 mm
- net /Project Architecture/Cell Sense & Balance/VC4: track 32.7 -> 35.9 mm
- net /Project Architecture/Cell Sense & Balance/VC3: track 30.7 -> 33.7 mm
- net /Project Architecture/Cell Sense & Balance/CB8: track 0.00 -> 1.50 mm
- net /Project Architecture/GND: vias 11 -> 36

Commit message: SCH[Connector]: Updated tap, and temp connectors to two row variants for space, combined grounds to one pin for the temp assuming the battery interface board combines those grounds.
Parts:
- removed the J4 at (93.8, 95.3)
- removed the J4 at (76.2, 102.3)
- added J4: 0430451024, remote_0430451024:CONN_SD-43045-009_10_MOL, F.Cu at (160.4, 70.9)
- J3: value 0430451612 -> 0430451200; footprint remote_0430451612:CONN_SD-43045-005_16_MOL -> remote_0430451200:CONN_SD-43045-001_12_MOL
- moved FID3 87.6 mm to (167.0, 68.8)
- moved FID2 62.5 mm to (167.0, 106.5)
- moved J3 52.3 mm to (107.0, 95.0), turned to -90 degrees
- moved FID1 24.5 mm to (108.0, 106.2)
- moved C28 8.93 mm to (113.8, 53.5)
- moved R20 8.93 mm to (108.5, 56.2)
- moved R21 8.93 mm to (113.3, 56.2)
- moved Q1 8.93 mm to (120.9, 55.0)
- moved C29 7.63 mm to (138.2, 76.7)
- moved C30 7.63 mm to (143.2, 76.7)
- moved C32 7.63 mm to (150.2, 76.7)
- moved C33 7.63 mm to (152.0, 76.7)
- moved C34 7.63 mm to (157.1, 76.7)
- moved C36 7.63 mm to (164.0, 76.7)
- moved R23 7.63 mm to (140.0, 75.6)
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Connections:
- J3 pad 1: /Project Architecture/Connectors/T_P8 -> /Project Architecture/VMODULE
- J3 pad 10: /Project Architecture/GND -> /Project Architecture/Cell Sense & Balance/TAP1
- J3 pad 11: /Project Architecture/GND -> /Project Architecture/Cell Sense & Balance/TAP0
- J3 pad 2: /Project Architecture/Connectors/T_P7 -> unconnected-(J3-Pad2)
- J3 pad 3: /Project Architecture/Connectors/T_P6 -> /Project Architecture/Cell Sense & Balance/TAP8
- J3 pad 4: /Project Architecture/Connectors/T_P5 -> /Project Architecture/Cell Sense & Balance/TAP7
- J3 pad 5: /Project Architecture/Connectors/T_P4 -> /Project Architecture/Cell Sense & Balance/TAP6
- J3 pad 6: /Project Architecture/Connectors/T_P3 -> /Project Architecture/Cell Sense & Balance/TAP5
- J3 pad 7: /Project Architecture/Connectors/T_P2 -> /Project Architecture/Cell Sense & Balance/TAP4
- J3 pad 8: /Project Architecture/Connectors/T_P1 -> /Project Architecture/Cell Sense & Balance/TAP3
- J3 pad 9: /Project Architecture/GND -> /Project Architecture/Cell Sense & Balance/TAP2
Routing:
- net /Project Architecture/Cell Sense & Balance/VC8: track 46.6 -> 5.40 mm
- net /Project Architecture/Cell Sense & Balance/VC7: track 43.6 -> 6.46 mm
- net /Project Architecture/Cell Sense & Balance/VC6: track 40.8 -> 6.23 mm
- net /Project Architecture/Cell Sense & Balance/VC5: track 38.2 -> 6.00 mm
- net /Project Architecture/Cell Sense & Balance/VC4: track 35.9 -> 5.77 mm
- net /Project Architecture/Cell Sense & Balance/VC3: track 33.7 -> 5.75 mm
- net /Project Architecture/Cell Sense & Balance/VC2: track 31.6 -> 5.98 mm
- net /Project Architecture/Cell Sense & Balance/VC0: track 35.9 -> 10.5 mm
- net /Project Architecture/Cell Sense & Balance/VC1: track 32.5 -> 7.64 mm
- net /Project Architecture/VMODULE: track 0.00 -> 22.0 mm
- net /Project Architecture/Cell Sense & Balance/TAP0: track 0.00 -> 20.1 mm
- net /Project Architecture/Cell Sense & Balance/TAP7: track 8.42 -> 24.5 mm
- net /Project Architecture/Cell Sense & Balance/TAP8: track 8.42 -> 23.9 mm
- net /Project Architecture/Cell Sense & Balance/TAP5: track 8.42 -> 16.5 mm
- net /Project Architecture/Cell Sense & Balance/TAP2: track 8.42 -> 15.9 mm
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