File: bms_slave.kicad_pcb (KiCad board)
At the start: 4 copper layers, 80 x 45 mm, 108 parts, among them J3 0430450200, J4 0436500200, J5 IPS1-110-01-L-D, Q1 ZXTN4004KQTC, U1 BQ79616PAPRQ1, U2 SM91502ALA-E, U3 SM91502ALA-E

Commit message: PCB[Grounding, Heat]: Added some more pours for heat considerations for bjt, stiched more vias for heat consideration on balanace resistors. SCH[Notes, Block Diagram]: Working on spelling and notes updates, started block diagram.
Parts:
- added H2: MountingHole, MountingHole:MountingHole_3.2mm_M3, F.Cu at (178.5, 106.0)
- added H5: MountingHole, MountingHole:MountingHole_3.2mm_M3, F.Cu at (178.5, 69.0)
- moved C28 0.79 mm to (132.8, 80.0), turned to -90 degrees
- renumbered C39 to C37, C40 to C38, C37 to C39, C38 to C40, C42 to C41, C41 to C42, CR2 to CR1, CR1 to CR2, FID3 to FID2, FID2 to FID3, H5 to H3, H2 to H4, J4 to J1, J3 to J2, J5 to J3, R40 to R39, R39 to R40, R43 to R41, R44 to R42, R41 to R43, R42 to R44, U3 to U2, U2 to U3
Routing:
- net /Project Architecture/Power & Reference/VCOLL: track 12.4 -> 1.84 mm
- net /Project Architecture/GND: vias 198 -> 228
- added copper zone on F.Cu, net /Project Architecture/Power & Reference/VCOLL
