File: bms_slave.kicad_pcb (KiCad board)
At the start: 4 copper layers, 80 x 45 mm, 131 parts, among them J1 0436500200, J2 0430450200, J3 IPS1-110-01-L-D, Q1 ZXTN4004KQTC, U1 BQ79616PAPRQ1, U2 SM91502ALA-E, U3 SM91502ALA-E

Commit message: PCB[Trace Size, Testpad, Daisy]: Changed Bat Trace size FAT, Made test pads larger, small trace movement to clean up, daisy trace change. SCH[Notes]: Small notes changes.
Parts:
- TP1, TP10, TP11, TP12, TP13, TP14, TP15, TP16, TP17, TP18, TP19, TP2, TP20, TP3, TP4, TP5, TP6, TP7, TP8, TP9: footprint TestPoint:TestPoint_Pad_1.0x1.0mm -> TestPoint:TestPoint_Pad_1.5x1.5mm
- moved TP11 0.30 mm to (107.2, 75.8)
- moved TP12 0.30 mm to (107.2, 78.4)
- moved TP13 0.30 mm to (107.2, 80.9)
- moved TP14 0.30 mm to (107.2, 83.4)
- moved TP15 0.30 mm to (107.2, 86.0)
- moved TP16 0.30 mm to (107.2, 88.5)
- moved TP17 0.30 mm to (107.2, 91.1)
- moved TP18 0.30 mm to (107.2, 93.6)
- moved TP19 0.30 mm to (107.2, 96.1)
- moved TP20 0.30 mm to (107.2, 98.7)
- moved TP1 0.20 mm to (113.7, 75.8)
- moved TP6 0.20 mm to (113.7, 88.5)
- moved TP8 0.20 mm to (113.7, 93.6)
- moved TP10 0.20 mm to (113.7, 98.7)
- moved TP2 0.20 mm to (113.7, 78.4)
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Routing:
- net /Project Architecture/Cell Sense & Balance/BAT: track 14.1 -> 2.21 mm
- net /Project Architecture/Connectors/COMH.P: track 6.35 -> 4.27 mm
- net /Project Architecture/VMODULE: track 43.6 -> 44.6 mm
- net /Project Architecture/GND: track 26.4 -> 26.9 mm, vias 228 -> 225
- added copper zone on F.Cu, net /Project Architecture/Cell Sense & Balance/BAT
