File: bms_slave.kicad_sch (KiCad schematic)
At the start: 0 parts

Commit message: SCH[Power & Balance]: Inital Schamtic for two pages.
Other:
- removed sheet Power - Sequencing
Changed lines of the file:
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@@
-	)
-	(sheet
-		(at 340.36 313.69)
-		(size 35.56 5.08)
-		(exclude_from_sim no)
-		(in_bom yes)
-		(on_board yes)
-		(dnp no)
-		(stroke
-			(width 0.1524)
-			(type solid)
-		)
-		(fill
-			(color 0 0 0 0)
-		)
-		(property "Sheetname" "Power - Sequencing"
-			(at 340.36 312.6609 0)
-			(show_name no)
-			(do_not_autoplace no)
-			(effects
-				(font
-					(face "Times New Roman")
-					(size 1.905 1.905)
-					(bold yes)
-					(color 0 0 0 1)
-				)
-				(justify left bottom)
-			)
-		)
-		(property "Sheetfile" "Power - Sequencing.kicad_sch"
-			(at 341.63 314.96 0)
-			(show_name no)
-			(do_not_autoplace no)
-			(effects
-				(font
-					(face "Arial")
-					(size 1.27 1.27)
-				)
-				(justify left top)
-			)
-		)
-		(instances
-			(project "bms_slave"
-				(path "/f9e05184-c88b-4a88-ae9c-ab2bdb32be7c"
-					(page "6")
-				)
-			)
-		)
 	)
 	(sheet
@@
 			(project "bms_slave"
 				(path "/f9e05184-c88b-4a88-ae9c-ab2bdb32be7c"
-					(page "7")
+					(page "11")
 				)
 			)

Commit message: PCB[Test Points, Mechanical, Silk]: Finalized Mounting Points, Added Testpoints with adjecent silkscreen labels. SCH[Test Points, Notes]: Added/Updated notes for all pages, cleaned up errors spelling ect.
Other:
- note added: "${PROJECT_NAME}"
- note added: "TI BQ79616PAPRQ1 Datasheet"
- note removed: "${BOARD_NAME}"
- note removed: "Comment"
- note removed: "Date: ${RELEASE_DATE}"
Changed lines of the file:
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@@
-		)
-	)
-	(text "Date: ${RELEASE_DATE}"
-		(exclude_from_sim no)
-		(at 220.98 237.49 0)
-		(effects
-			(font
-				(face "Times New Roman")
-				(size 10.16 10.16)
-				(thickness 0.6)
-				(bold yes)
-				(color 200 200 200 1)
-			)
-			(justify left bottom)
 		)
 	)
@@
 		)
 	)
-	(text "${BOARD_NAME}"
+	(text "${PROJECT_NAME}"
 		(exclude_from_sim no)
 		(at 25.4 40.64 0)
@@
 		)
 	)
-	(text "Comment"
+	(text "TI BQ79616PAPRQ1 Datasheet"
 		(exclude_from_sim no)
 		(at 222.25 177.8 0)
@@
 			)
 			(justify left bottom)
-		)
-	)
+			(href "https://www.ti.com/lit/ds/symlink/bq79612-q1.pdf")
+		)
+	)
